File: EAGLE Files/OMNIBUS Stepper board v3.brd (EAGLE design)
At the start: 100.6 x 73.6 mm, 52 parts, among them K7 691131710005, K8 691131710005, K9 691131710005, Q1 BTS134D, U2 L7805ACD2T-TR

Commit message: new DRV board version and updates
Parts:
- removed C6: 0.33uf 50v, rcl:C1206
- removed C7: 100nf, rcl:C0805
- removed D2: SS310, SS54:DO-214AC
- removed EN-LOW: (no value), pinhead:1X02
- removed LASER-ON: blue, led:CHIPLED_0805
- removed MIC2954: MIC2954, MIC2954:SOT223
- removed Q1: BTS134D, FQD7N10LTM:TO-252
- added EN: (no value), pinhead:1X02
- added JP5, JP6, JP7, JP8: (no value), pinhead:1X01
- added Q3: FQD7N10LTM, FQD7N10LTM:TO-252
- added R8: 10k, rcl:R0805
- added U1: CJ78M05-1300040P1, CJ78M05:TO252
- R1: value 1k -> 220
- R2: value 10k -> 100
- R3: value 470 -> 1k
- U2: value L7805ACD2T-TR -> PC817X3NSZ1B; device L7805ACD2T-TR:TO254P1515X470-3N -> PC817X3NSZ1B:DIP762W50P254L495H455Q4
- moved U2 36.9 mm to (51.2, 50.9), turned to 270 degrees
- moved J1 22.9 mm to (71.1, 49.5)
- moved R3 18.1 mm to (51.1, 57.4)
- moved R2 16.6 mm to (59.3, 55.9), turned to 180 degrees
- moved R1 11.7 mm to (47.0, 50.8), turned to 90 degrees
- moved C9 9.44 mm to (38.4, 46.9)
- moved C4 2.95 mm to (38.1, 57.1), turned to 0 degrees
- moved R4 2.54 mm to (22.9, 49.5)
- moved R5 2.54 mm to (22.9, 52.8)
- moved D4 1.27 mm to (27.2, 64.3)
- moved JP_Y 0.38 mm to (57.1, 41.5)
- moved JP_X 0.25 mm to (31.8, 41.7)
- moved JP_Z 0.25 mm to (82.5, 41.7)
Connections:
- removed net GND_SW: D2.A, J1.3
- removed net L_SW: D2.C, LASER-ON.C, Q1.T
- new net N$4: R2.2, R3.1, U2.3
- new net NEG_LOAD: J1.3, Q3.T
- net 12V_BD: now also JP8.1; no longer C4.1, C7.2, MIC2954.1, U2.2
- net 12V_LASER: now also U2.4; no longer R1.1
- net 5V: now also U1.3; no longer MIC2954.3
- net 5VPWM: now also R1.2; no longer R3.2
- net EN: now also EN.2; no longer EN-LOW.2
- net GND: now also EN.1, JP6.1, JP7.1, Q3.3, R3.2, R8.2, U1.2, U2.2; no longer C6.2, C7.1, EN-LOW.1, MIC2954.2, MIC2954.4, Q1.3, R2.2, U2.3
- net N$1: now also Q3.1, R8.1; no longer Q1.1, R3.1
- net N$3: now also R1.1, U2.1; no longer LASER-ON.A, R1.2
- net RAW_2: now also C4.1, JP5.1, U1.1; no longer C6.1, U2.1
Routing:
- net 12V_BD: track 53.2 -> 25.1 mm
- net L_SW: track 19.3 -> 0.00 mm
- net N$4: track 0.00 -> 18.4 mm
- net 5VPWM: track 39.6 -> 56.0 mm
- net 12V_LASER: track 30.5 -> 46.6 mm, vias 1 -> 0
- net GND_SW: track 9.93 -> 0.00 mm
- net NEG_LOAD: track 0.00 -> 8.76 mm
- net RAW_2: track 274.6 -> 279.9 mm
- net N$3: track 2.84 -> 8.08 mm
- net X_DIR: track 64.5 -> 69.3 mm
- net 5V: track 289.1 -> 284.7 mm
- net Y_DIR: track 53.0 -> 57.4 mm
- net N$7: track 11.5 -> 9.11 mm
- net GND: track 7.62 -> 9.92 mm, vias 31 -> 32
- net N$2: track 7.19 -> 5.10 mm
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Other:
- board text added: "G"
- board text added: "iFLIGHT 12V 2A StepDown #1"
- board text added: "iFLIGHT 12V 2A StepDown #2 (LSR)"
- board text removed: "iFLIGHT 12V 2A Laser StepDown"
