File: EAGLE Files/OMNIBUS Stepper board v3.sch (EAGLE design)
At the start: 52 parts, among them K7 691131710005, K8 691131710005, K9 691131710005, Q1 BTS134D, U2 L7805ACD2T-TR

Commit message: new DRV board version and updates
Parts:
- removed C6: 0.33uf 50v, rcl:C-EUC1206
- removed C7: 100nf, rcl:C-EUC0805
- removed D2: SS310, SS54:SS54
- removed LASER-ON: blue, led:LEDCHIPLED_0805
- removed MIC2954: MIC2954, MIC2954:MIC2954
- removed Q1: BTS134D, FQD7N10LTM:FQD7N10LTM
- added JP5, JP6, JP7, JP8: (no value), pinhead:PINHD-1X1
- added Q3: FQD7N10LTM, FQD7N10LTM:FQD7N10LTM
- added R8: 10k, rcl:R-EU_R0805
- added U1: CJ78M05-1300040P1, CJ78M05:CJ78M05-1300040P1
- R1: value 1k -> 220
- R2: value 10k -> 100
- R3: value 470 -> 1k
- U2: value L7805ACD2T-TR -> PC817X3NSZ1B; device L7805ACD2T-TR:L7805ACD2T-TR -> PC817X3NSZ1B:PC817X3NSZ1B
- renumbered EN-LOW to EN
Connections:
- removed net GND_SW: D2.A, J1.3
- removed net L_SW: D2.C, LASER-ON.C, Q1.D
- new net N$4: R2.2, R3.1, U2.EMITTER
- new net NEG_LOAD: J1.3, Q3.D
- net 12V_BD: now also JP8.1; no longer C4.1, C7.2, MIC2954.IN, U2.OUT
- net 12V_LASER: now also U2.COLLECTOR; no longer R1.1
- net 5V: now also U1.OUT; no longer MIC2954.OUT
- net 5VPWM: now also R1.2; no longer R3.2
- net GND: now also JP6.1, JP7.1, Q3.S, R3.2, R8.2, U1.GND, U2.CATHODE; no longer C6.2, C7.1, MIC2954.GND@0, MIC2954.GND@1, Q1.S, R2.2, U2.GND
- net N$1: now also Q3.G, R8.1; no longer Q1.G, R3.1
- net N$3: now also R1.1, U2.ANODE; no longer LASER-ON.A, R1.2
- net RAW_2: now also C4.1, JP5.1, U1.IN; no longer C6.1, U2.IN
Other:
- moved on the sheet: R1, R2, R3
